Commit message: [tiago] Lump gripper inertia into arm dynamics

File: gato/dynamics/tiago_right/tiago_right_arm_include_gripper.urdf (robot description, URDF)
Before this commit: robot tiago_pro_right_arm, 9 links, 8 joints
Links:
- added link gripper_right_base_link, mass 0.59671873; collision mesh filename=package://pal_pro_gripper_description/meshes/base_link_tc.s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; visual mesh filename=package://pal_pro_gripper_description/meshes/base_link_tc.s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
- added link gripper_right_fingertip_left_link, mass 0.0335029606041878; collision mesh filename=package://pal_pro_gripper_description/meshes/fingertip.stl; visual mesh filename=package://pal_pro_gripper_description/meshes/fingertip.stl
- added link gripper_right_fingertip_right_link, mass 0.0335029606041878; collision mesh filename=package://pal_pro_gripper_description/meshes/fingertip.stl; visual mesh filename=package://pal_pro_gripper_description/meshes/fingertip.stl
- added link gripper_right_inner_finger_left_link, mass 0.018619; collision mesh filename=package://pal_pro_gripper_description/meshes/inner_finger.s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; visual mesh filename=package://pal_pro_gripper_description/meshes/inner_finger.s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
- added link gripper_right_inner_finger_right_link, mass 0.018619; collision mesh filename=package://pal_pro_gripper_description/meshes/inner_finger.s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; visual mesh filename=package://pal_pro_gripper_description/meshes/inner_finger.s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
- added link gripper_right_outer_finger_left_link, mass 0.0159887772377711; collision mesh filename=package://pal_pro_gripper_description/meshes/outer_finger.s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; visual mesh filename=package://pal_pro_gripper_description/meshes/outer_finger.s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
- added link gripper_right_outer_finger_right_link, mass 0.0159887772377711; collision mesh filename=package://pal_pro_gripper_description/meshes/outer_finger.s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; visual mesh filename=package://pal_pro_gripper_description/meshes/outer_finger.s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
- link arm_right_tool_link: mass 0.73294020568391793 -> None
Joints:
- added joint gripper_right_base_joint: type fixed, parent arm_right_tool_link, child gripper_right_base_link, origin xyz=0.0 0.0 0.0 rpy=0 0 0, axis 0 0 0
- added joint gripper_right_finger_joint: type revolute, parent gripper_right_base_link, child gripper_right_outer_finger_left_link, origin xyz=0 -0.0288 0.0743 rpy=1.5708 0.83776 -1.5708, axis 0 0 1, limit lower=0 upper=0.8028514559173916 effort=0.1 velocity=2
- added joint gripper_right_fingertip_left_joint: type revolute, parent gripper_right_inner_finger_left_link, child gripper_right_fingertip_left_link, origin xyz=0 0.05 0 rpy=0 0 0.83776, axis 0 0 1, limit lower=-0.8028514559173916 upper=0 effort=0.1 velocity=2, mimic joint=gripper_right_finger_joint multiplier=-1 offset=0
- added joint gripper_right_fingertip_right_joint: type revolute, parent gripper_right_inner_finger_right_link, child gripper_right_fingertip_right_link, origin xyz=0 0.05 0 rpy=0 0 0.83776, axis 0 0 1, limit lower=-0.8028514559173916 upper=0 effort=0.1 velocity=2, mimic joint=gripper_right_finger_joint multiplier=-1 offset=0
- added joint gripper_right_inner_finger_left_joint: type revolute, parent gripper_right_base_link, child gripper_right_inner_finger_left_link, origin xyz=0 -0.013977 0.078832 rpy=1.5708 0.83776 -1.5708, axis 0 0 1, limit lower=0 upper=0.8028514559173916 effort=0.1 velocity=2, mimic joint=gripper_right_finger_joint multiplier=1 offset=0
- added joint gripper_right_inner_finger_right_joint: type revolute, parent gripper_right_base_link, child gripper_right_inner_finger_right_link, origin xyz=0 0.013977 0.078832 rpy=1.5708 0.83776 1.5708, axis 0 0 1, limit lower=0 upper=0.8028514559173916 effort=0.1 velocity=2, mimic joint=gripper_right_finger_joint multiplier=1 offset=0
- added joint gripper_right_outer_finger_right_joint: type revolute, parent gripper_right_base_link, child gripper_right_outer_finger_right_link, origin xyz=0 0.0288 0.0743 rpy=1.5708 0.83776 1.5708, axis 0 0 1, limit lower=0 upper=0.8028514559173916 effort=0.1 velocity=2, mimic joint=gripper_right_finger_joint multiplier=1 offset=0
